Commit message: corrected digit_model.urdf mesh paths

File: urdf/digit_model.urdf (robot description, URDF)
Before this commit: robot digit, 29 links, 28 joints
Links:
- link left_elbow: geometry collision mesh filename=arm-L4.obj; visual mesh filename=arm-L4.obj
- link left_hip_pitch: geometry collision mesh filename=hip-pitch.obj; visual mesh filename=hip-pitch.obj
- link left_hip_roll: geometry collision mesh filename=hip-yaw-housing.obj; visual mesh filename=hip-yaw-housing.obj
- link left_hip_yaw: geometry collision mesh filename=hip-pitch-housing.obj; visual mesh filename=hip-pitch-housing.obj
- link left_knee: geometry collision mesh filename=knee.obj; visual mesh filename=knee.obj
- link left_shin: geometry collision mesh filename=shin.obj; visual mesh filename=shin.obj
- link left_shoulder_cap: geometry collision mesh filename=shoulder-roll-housing.obj; visual mesh filename=shoulder-roll-housing.obj
- link left_shoulder_pitch: geometry collision mesh filename=arm-L2.obj; visual mesh filename=arm-L2.obj
- link left_shoulder_roll: geometry collision mesh filename=arm-L1.obj; visual mesh filename=arm-L1.obj
- link left_shoulder_yaw: geometry collision mesh filename=arm-L3.obj; visual mesh filename=arm-L3.obj
- link left_tarsus: geometry collision mesh filename=tarsus.obj; visual mesh filename=tarsus.obj
- link left_toe_pitch: geometry collision mesh filename=toe-pitch.obj; visual mesh filename=toe-pitch.obj
- link left_toe_roll: geometry collision mesh filename=toe-roll.obj; visual mesh filename=toe-roll.obj
- link left_waist_cap: geometry collision mesh filename=shoulder-roll-housing.obj; visual mesh filename=shoulder-roll-housing.obj
- link right_elbow: geometry collision mesh filename=arm-L4.obj scale=1 -1 1; visual mesh filename=arm-L4.obj scale=1 -1 1
- link right_hip_pitch: geometry collision mesh filename=hip-pitch.obj scale=1 -1 1; visual mesh filename=hip-pitch.obj scale=1 -1 1
- link right_hip_roll: geometry collision mesh filename=hip-yaw-housing.obj scale=1 -1 1; visual mesh filename=hip-yaw-housing.obj scale=1 -1 1
- link right_hip_yaw: geometry collision mesh filename=hip-pitch-housing.obj scale=1 -1 1; visual mesh filename=hip-pitch-housing.obj scale=1 -1 1
- link right_knee: geometry collision mesh filename=knee.obj scale=1 -1 1; visual mesh filename=knee.obj scale=1 -1 1
- link right_shin: geometry collision mesh filename=shin.obj scale=1 -1 1; visual mesh filename=shin.obj scale=1 -1 1
- link right_shoulder_cap: geometry collision mesh filename=shoulder-roll-housing.obj scale=1 -1 1; visual mesh filename=shoulder-roll-housing.obj scale=1 -1 1
- link right_shoulder_pitch: geometry collision mesh filename=arm-L2.obj scale=1 -1 1; visual mesh filename=arm-L2.obj scale=1 -1 1
- link right_shoulder_roll: geometry collision mesh filename=arm-L1.obj scale=1 -1 1; visual mesh filename=arm-L1.obj scale=1 -1 1
- link right_shoulder_yaw: geometry collision mesh filename=arm-L3.obj scale=1 -1 1; visual mesh filename=arm-L3.obj scale=1 -1 1
- link right_tarsus: geometry collision mesh filename=tarsus.obj scale=1 -1 1; visual mesh filename=tarsus.obj scale=1 -1 1
- link right_toe_pitch: geometry collision mesh filename=toe-pitch.obj scale=1 -1 1; visual mesh filename=toe-pitch.obj scale=1 -1 1
- link right_toe_roll: geometry collision mesh filename=toe-roll.obj scale=1 -1 1; visual mesh filename=toe-roll.obj scale=1 -1 1
- link right_waist_cap: geometry collision mesh filename=shoulder-roll-housing.obj scale=1 -1 1; visual mesh filename=shoulder-roll-housing.obj scale=1 -1 1
- link torso: geometry collision mesh filename=torso.obj; visual mesh filename=torso.obj

Commit message: corrected digit_model.urdf

File: urdf/digit_model.urdf (robot description, URDF)
Before this commit: robot digit, 29 links, 28 joints
Links:
- link left_elbow: geometry collision mesh filename=urdf/arm-L4.obj; visual mesh filename=urdf/arm-L4.obj
- link left_hip_pitch: geometry collision mesh filename=urdf/hip-pitch.obj; visual mesh filename=urdf/hip-pitch.obj
- link left_hip_roll: geometry collision mesh filename=urdf/hip-yaw-housing.obj; visual mesh filename=urdf/hip-yaw-housing.obj
- link left_hip_yaw: geometry collision mesh filename=urdf/hip-pitch-housing.obj; visual mesh filename=urdf/hip-pitch-housing.obj
- link left_knee: geometry collision mesh filename=urdf/knee.obj; visual mesh filename=urdf/knee.obj
- link left_shin: geometry collision mesh filename=urdf/shin.obj; visual mesh filename=urdf/shin.obj
- link left_shoulder_cap: geometry collision mesh filename=urdf/shoulder-roll-housing.obj; visual mesh filename=urdf/shoulder-roll-housing.obj
- link left_shoulder_pitch: geometry collision mesh filename=urdf/arm-L2.obj; visual mesh filename=urdf/arm-L2.obj
- link left_shoulder_roll: geometry collision mesh filename=urdf/arm-L1.obj; visual mesh filename=urdf/arm-L1.obj
- link left_shoulder_yaw: geometry collision mesh filename=urdf/arm-L3.obj; visual mesh filename=urdf/arm-L3.obj
- link left_tarsus: geometry collision mesh filename=urdf/tarsus.obj; visual mesh filename=urdf/tarsus.obj
- link left_toe_pitch: geometry collision mesh filename=urdf/toe-pitch.obj; visual mesh filename=urdf/toe-pitch.obj
- link left_toe_roll: geometry collision mesh filename=urdf/toe-roll.obj; visual mesh filename=urdf/toe-roll.obj
- link left_waist_cap: geometry collision mesh filename=urdf/shoulder-roll-housing.obj; visual mesh filename=urdf/shoulder-roll-housing.obj
- link right_elbow: geometry collision mesh filename=urdf/arm-L4.obj scale=1 -1 1; visual mesh filename=urdf/arm-L4.obj scale=1 -1 1
- link right_hip_pitch: geometry collision mesh filename=urdf/hip-pitch.obj scale=1 -1 1; visual mesh filename=urdf/hip-pitch.obj scale=1 -1 1
- link right_hip_roll: geometry collision mesh filename=urdf/hip-yaw-housing.obj scale=1 -1 1; visual mesh filename=urdf/hip-yaw-housing.obj scale=1 -1 1
- link right_hip_yaw: geometry collision mesh filename=urdf/hip-pitch-housing.obj scale=1 -1 1; visual mesh filename=urdf/hip-pitch-housing.obj scale=1 -1 1
- link right_knee: geometry collision mesh filename=urdf/knee.obj scale=1 -1 1; visual mesh filename=urdf/knee.obj scale=1 -1 1
- link right_shin: geometry collision mesh filename=urdf/shin.obj scale=1 -1 1; visual mesh filename=urdf/shin.obj scale=1 -1 1
- link right_shoulder_cap: geometry collision mesh filename=urdf/shoulder-roll-housing.obj scale=1 -1 1; visual mesh filename=urdf/shoulder-roll-housing.obj scale=1 -1 1
- link right_shoulder_pitch: geometry collision mesh filename=urdf/arm-L2.obj scale=1 -1 1; visual mesh filename=urdf/arm-L2.obj scale=1 -1 1
- link right_shoulder_roll: geometry collision mesh filename=urdf/arm-L1.obj scale=1 -1 1; visual mesh filename=urdf/arm-L1.obj scale=1 -1 1
- link right_shoulder_yaw: geometry collision mesh filename=urdf/arm-L3.obj scale=1 -1 1; visual mesh filename=urdf/arm-L3.obj scale=1 -1 1
- link right_tarsus: geometry collision mesh filename=urdf/tarsus.obj scale=1 -1 1; visual mesh filename=urdf/tarsus.obj scale=1 -1 1
- link right_toe_pitch: geometry collision mesh filename=urdf/toe-pitch.obj scale=1 -1 1; visual mesh filename=urdf/toe-pitch.obj scale=1 -1 1
- link right_toe_roll: geometry collision mesh filename=urdf/toe-roll.obj scale=1 -1 1; visual mesh filename=urdf/toe-roll.obj scale=1 -1 1
- link right_waist_cap: geometry collision mesh filename=urdf/shoulder-roll-housing.obj scale=1 -1 1; visual mesh filename=urdf/shoulder-roll-housing.obj scale=1 -1 1
- link torso: geometry collision mesh filename=urdf/torso.obj; visual mesh filename=urdf/torso.obj

Commit message: corrected digit_model.urdf

File: urdf/digit_model.urdf (robot description, URDF)
Before this commit: robot digit, 29 links, 28 joints
Links:
- link left_elbow: geometry collision mesh filename=package://urdf/arm-L4.obj; visual mesh filename=package://urdf/arm-L4.obj
- link left_hip_pitch: geometry collision mesh filename=package://urdf/hip-pitch.obj; visual mesh filename=package://urdf/hip-pitch.obj
- link left_hip_roll: geometry collision mesh filename=package://urdf/hip-yaw-housing.obj; visual mesh filename=package://urdf/hip-yaw-housing.obj
- link left_hip_yaw: geometry collision mesh filename=package://urdf/hip-pitch-housing.obj; visual mesh filename=package://urdf/hip-pitch-housing.obj
- link left_knee: geometry collision mesh filename=package://urdf/knee.obj; visual mesh filename=package://urdf/knee.obj
- link left_shin: geometry collision mesh filename=package://urdf/shin.obj; visual mesh filename=package://urdf/shin.obj
- link left_shoulder_cap: geometry collision mesh filename=package://urdf/shoulder-roll-housing.obj; visual mesh filename=package://urdf/shoulder-roll-housing.obj
- link left_shoulder_pitch: geometry collision mesh filename=package://urdf/arm-L2.obj; visual mesh filename=package://urdf/arm-L2.obj
- link left_shoulder_roll: geometry collision mesh filename=package://urdf/arm-L1.obj; visual mesh filename=package://urdf/arm-L1.obj
- link left_shoulder_yaw: geometry collision mesh filename=package://urdf/arm-L3.obj; visual mesh filename=package://urdf/arm-L3.obj
- link left_tarsus: geometry collision mesh filename=package://urdf/tarsus.obj; visual mesh filename=package://urdf/tarsus.obj
- link left_toe_pitch: geometry collision mesh filename=package://urdf/toe-pitch.obj; visual mesh filename=package://urdf/toe-pitch.obj
- link left_toe_roll: geometry collision mesh filename=package://urdf/toe-roll.obj; visual mesh filename=package://urdf/toe-roll.obj
- link left_waist_cap: geometry collision mesh filename=package://urdf/shoulder-roll-housing.obj; visual mesh filename=package://urdf/shoulder-roll-housing.obj
- link right_elbow: geometry collision mesh filename=package://urdf/arm-L4.obj scale=1 -1 1; visual mesh filename=package://urdf/arm-L4.obj scale=1 -1 1
- link right_hip_pitch: geometry collision mesh filename=package://urdf/hip-pitch.obj scale=1 -1 1; visual mesh filename=package://urdf/hip-pitch.obj scale=1 -1 1
- link right_hip_roll: geometry collision mesh filename=package://urdf/hip-yaw-housing.obj scale=1 -1 1; visual mesh filename=package://urdf/hip-yaw-housing.obj scale=1 -1 1
- link right_hip_yaw: geometry collision mesh filename=package://urdf/hip-pitch-housing.obj scale=1 -1 1; visual mesh filename=package://urdf/hip-pitch-housing.obj scale=1 -1 1
- link right_knee: geometry collision mesh filename=package://urdf/knee.obj scale=1 -1 1; visual mesh filename=package://urdf/knee.obj scale=1 -1 1
- link right_shin: geometry collision mesh filename=package://urdf/shin.obj scale=1 -1 1; visual mesh filename=package://urdf/shin.obj scale=1 -1 1
- link right_shoulder_cap: geometry collision mesh filename=package://urdf/shoulder-roll-housing.obj scale=1 -1 1; visual mesh filename=package://urdf/shoulder-roll-housing.obj scale=1 -1 1
- link right_shoulder_pitch: geometry collision mesh filename=package://urdf/arm-L2.obj scale=1 -1 1; visual mesh filename=package://urdf/arm-L2.obj scale=1 -1 1
- link right_shoulder_roll: geometry collision mesh filename=package://urdf/arm-L1.obj scale=1 -1 1; visual mesh filename=package://urdf/arm-L1.obj scale=1 -1 1
- link right_shoulder_yaw: geometry collision mesh filename=package://urdf/arm-L3.obj scale=1 -1 1; visual mesh filename=package://urdf/arm-L3.obj scale=1 -1 1
- link right_tarsus: geometry collision mesh filename=package://urdf/tarsus.obj scale=1 -1 1; visual mesh filename=package://urdf/tarsus.obj scale=1 -1 1
- link right_toe_pitch: geometry collision mesh filename=package://urdf/toe-pitch.obj scale=1 -1 1; visual mesh filename=package://urdf/toe-pitch.obj scale=1 -1 1
- link right_toe_roll: geometry collision mesh filename=package://urdf/toe-roll.obj scale=1 -1 1; visual mesh filename=package://urdf/toe-roll.obj scale=1 -1 1
- link right_waist_cap: geometry collision mesh filename=package://urdf/shoulder-roll-housing.obj scale=1 -1 1; visual mesh filename=package://urdf/shoulder-roll-housing.obj scale=1 -1 1
- link torso: geometry collision mesh filename=package://urdf/torso.obj; visual mesh filename=package://urdf/torso.obj
